File: kicad/218-pdb.kicad_pcb (KiCad board)
At the start: 2 copper layers, 80 x 55.4 mm, 75 parts, among them J1 Conn_01x03, J10 Conn_01x03, J11 Conn_01x03, J12 Conn_01x03, J13 Conn_01x03, J14 Conn_01x03, J15 Conn_01x03, J16 Conn_01x03, J17 Conn_01x03, J18 Conn_01x03, J19 Conn_01x03, J2 Conn_01x03, J20 Conn_01x03, J21 Conn_01x03, J22 Conn_01x03, J23 Conn_01x03, J24 Conn_01x03, J25 Conn_01x04_Pin, J26 Conn_01x04_Pin, J27 Conn_01x04_Pin, J28 Conn_01x04_Pin, J29 14 V molex, J3 Conn_01x03, J30 14 V molex, J31 14 V molex, J32 14 V molex, J33 external 5V, J34 battery, J35 battery, J4 Conn_01x03, J5 Conn_01x03, J6 Conn_01x03, J7 Conn_01x03, J8 Conn_01x03, J9 Conn_01x03, SW1 5V switch, U3 LD1117V33, U4 LD1117V33

Commit message: draw traces, design B
Parts:
- removed FID2: jumper, 218-pdb:jumper
- removed NT3: ~, 218-pdb:PinHeader_1x03_P2.54mm_Vertical
- removed extSW1: switch, 218-pdb:Molex_KK-254_AE-6410-02A_1x02_P2.54mm_Vertical
- added D6: D, Diode_THT:D_DO-41_SOD81_P2.54mm_Vertical_AnodeUp, F.Cu at (145.2, 94.2)
- moved FID1 13.3 mm to (144.1, 80.6)
- moved R2 5.22 mm to (151.3, 75.2)
- moved R1 5.20 mm to (151.2, 64.6)
- moved D2 3.33 mm to (147.8, 75.2), turned to 180 degrees
- moved D1 3.29 mm to (147.8, 64.6), turned to 180 degrees
- moved R3 2.53 mm to (133.5, 88.8), turned to 180 degrees
- moved SW1 2.40 mm to (152.4, 85.3)
- moved D3 2.15 mm to (137.4, 93.3), turned to 180 degrees
- moved R4 1.79 mm to (148.6, 52.8), turned to -90 degrees
- moved R5 1.77 mm to (139.7, 52.8), turned to -90 degrees
- moved C5 0.40 mm to (142.4, 74.5)
- moved C4 0.11 mm to (142.2, 63.4)
Connections:
- SW1 pad 1: Net-(NT3-B) -> +BATT
Routing:
- net 5-2: track 0.00 -> 114.9 mm, vias 0 -> 6
- net 5-1: track 0.00 -> 109.3 mm
- net 14-3: track 0.00 -> 97.9 mm
- net +BATT: track 0.00 -> 97.5 mm
- net 3.3-2: track 0.00 -> 75.4 mm
- net 3.3-1: track 0.00 -> 69.9 mm
- net GND: track 0.00 -> 43.3 mm
- net 14-2: track 0.00 -> 40.0 mm
- net Net-(NT1-A): track 0.00 -> 33.2 mm, vias 0 -> 4
- net 14-1: track 0.00 -> 32.6 mm
- net Net-(J17-Pin_3): track 0.00 -> 13.6 mm
- net Net-(J1-Pin_3): track 0.00 -> 13.5 mm
- net Net-(J26-Pin_4): track 0.00 -> 12.3 mm
- net Net-(J24-Pin_3): track 0.00 -> 11.0 mm
- net Net-(J18-Pin_3): track 0.00 -> 8.48 mm
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Other:
- board text added: "5V"
- board text added: "motor"
