File: kicad/218-pdb.kicad_pcb (KiCad board)
At the start: 2 copper layers, 80 x 55.4 mm, 73 parts, among them J1 Conn_01x03, J10 Conn_01x03, J11 Conn_01x03, J12 Conn_01x03, J13 Conn_01x03, J14 Conn_01x03, J15 Conn_01x03, J16 Conn_01x03, J17 Conn_01x03, J18 Conn_01x03, J19 Conn_01x03, J2 Conn_01x03, J20 Conn_01x03, J21 Conn_01x03, J22 Conn_01x03, J23 Conn_01x03, J24 Conn_01x03, J25 Conn_01x04_Pin, J26 Conn_01x04_Pin, J27 Conn_01x04_Pin, J28 Conn_01x04_Pin, J29 14 V molex, J3 Conn_01x03, J30 14 V molex, J31 14 V molex, J32 14 V molex, J33 external 5V, J34 battery, J35 battery, J4 Conn_01x03, J5 Conn_01x03, J6 Conn_01x03, J7 Conn_01x03, J8 Conn_01x03, J9 Conn_01x03, SW1 5V switch, U1 DC-DC buck, U2 DC-DC buck, U3 LD1117V33, U4 LD1117V33

Commit message: cleanup
Other:
- board text added: "+"
- board text added: "+ - + -"
- board text added: "-"
- board text added: "Battery"
- board text removed: "Battery +- +-"
Changed lines of the file:
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@@
+	)
+	(gr_line
+		(start 138.938 89.662)
+		(end 137.414 85.598)
+		(stroke
+			(width 0.1)
+			(type default)
+		)
+		(layer "F.SilkS")
 	)
 	(gr_line
@@
 	)
 	(gr_line
+		(start 137.780754 85.964754)
+		(end 137.414 85.598)
+		(stroke
+			(width 0.1)
+			(type default)
+		)
+		(layer "F.SilkS")
+	)
+	(gr_line
 		(start 90.17 83.82)
 		(end 96.52 88.9)
@@
 	)
 	(gr_line
-		(start 140.927864 90.381864)
-		(end 135.780396 85.234396)
-		(stroke
-			(width 0.1)
-			(type default)
-		)
-		(layer "F.SilkS")
-	)
-	(gr_line
 		(start 93.98 53.34)
 		(end 82.55 58.42)
@@
 		(start 118.11 53.289529)
 		(end 113.03 58.42)
+		(stroke
+			(width 0.1)
+			(type default)
+		)
+		(layer "F.SilkS")
+	)
+	(gr_line
+		(start 137.414 85.598)
+		(end 137.414 86.106)
 		(stroke
 			(width 0.1)
@@
 	)
 	(gr_text "switch"
-		(at 152.4 78.359 0)
+		(at 152.373296 80.504479 0)
 		(layer "F.SilkS")
 		(effects
@@
 				(thickness 0.125)
 			)
+		)
+	)
+	(gr_text "+"
+		(at 138.9 83.82 0)
+		(layer "F.SilkS")
+		(effects
+			(font
+				(size 1.5 1.5)
+				(thickness 0.1875)
+			)
+			(justify left bottom)
 		)
 	)
@@
 		)
 	)
+	(gr_text "-"
+		(at 138.980647 88.100738 0)
+		(layer "F.SilkS")
+		(effects
+			(font
+				(size 1.5 1.5)
+				(thickness 0.1875)
+			)
+			(justify left bottom)
+		)
+	)
 	(gr_text "5\nG\n3"
 		(at 76.835 74.93 0)
@@
 		)
 	)
+	(gr_text "+   - +      -"
+		(at 85.337466 97.267084 0)
+		(layer "F.SilkS")
+		(effects
+			(font
+				(size 1.5 1.5)
+				(thickness 0.1875)
+			)
+			(justify left bottom)
+		)
+	)
 	(gr_text "v2.0\n2026"
 		(at 99.922898 94.60369 0)
@@
 		)
 	)
-	(gr_text "  Battery\n+- +-"
+	(gr_text "  Battery\n    "
 		(at 93.451157 97.408111 0)
 		(layer "F.SilkS")

Commit message: update script
Routing:
- net 14-3: track 97.9 -> 143.4 mm
- net GND: track 43.3 -> 54.2 mm
Other:
- board text added: "+ -"
