File: kicad/218-pdb.kicad_sch (KiCad schematic)
At the start: 67 parts, among them J1 Conn_01x03, J10 Conn_01x03, J11 Conn_01x03, J12 Conn_01x03, J13 Conn_01x03, J14 Conn_01x03, J15 Conn_01x03, J16 Conn_01x03, J17 Conn_01x03, J18 Conn_01x03, J19 Conn_01x03, J2 Conn_01x03, J20 Conn_01x03, J21 Conn_01x03, J22 Conn_01x03, J23 Conn_01x03, J24 Conn_01x03, J25 Conn_01x04_Pin, J26 Conn_01x04_Pin, J27 Conn_01x04_Pin, J28 Conn_01x04_Pin, J29 14 V molex, J3 Conn_01x03, J30 14 V molex, J31 14 V molex, J32 14 V molex, J33 external 5V, J34 battery, J35 battery, J4 Conn_01x03, J5 Conn_01x03, J6 Conn_01x03, J7 Conn_01x03, J8 Conn_01x03, J9 Conn_01x03, SW1 5V switch, U3 LD1117V33, U4 LD1117V33

Commit message: draw traces, design B
Parts:
- removed FID2: jumper, 218-pdb:jumper, symbol Mechanical:Fiducial
- removed NT3: ~, 218-pdb:PinHeader_1x03_P2.54mm_Vertical, symbol Switch:SW_SPDT
- removed extSW1: switch, 218-pdb:Molex_KK-254_AE-6410-02A_1x02_P2.54mm_Vertical, symbol Switch:SW_SPST
- added D6: D, Diode_THT:D_DO-41_SOD81_P2.54mm_Vertical_AnodeUp, symbol Device:D
Connections:
- net +BATT: now also SW1.1 (A)
- net 14-1: now also D6.1 (K)
- net 14-3: now also D6.2 (A)
Other:
- note added: "powered if either switch is on"
- moved on the sheet: D3, NT2, R3, SW1
