File: kicad/218-pdb.kicad_sch (KiCad schematic)
At the start: 73 parts, among them J1 Conn_01x03, J10 Conn_01x03, J11 Conn_01x03, J12 Conn_01x03, J13 Conn_01x03, J14 Conn_01x03, J15 Conn_01x03, J16 Conn_01x03, J17 Conn_01x03, J18 Conn_01x03, J19 Conn_01x03, J2 Conn_01x03, J20 Conn_01x03, J21 Conn_01x03, J22 Conn_01x03, J23 Conn_01x03, J24 Conn_01x03, J25 Conn_01x04_Pin, J26 Conn_01x04_Pin, J27 Conn_01x04_Pin, J28 Conn_01x04_Pin, J29 14 V molex, J3 Conn_01x03, J30 14 V molex, J31 14 V molex, J32 14 V molex, J33 external 5V, J34 battery, J35 battery, J4 Conn_01x03, J5 Conn_01x03, J6 Conn_01x03, J7 Conn_01x03, J8 Conn_01x03, J9 Conn_01x03, SW1 5V switch, U1 DC-DC buck, U2 DC-DC buck, U3 LD1117V33, U4 LD1117V33

Commit message: cleanup
Parts:
- FID10, FID3, FID4, FID5, FID6, FID7, FID8, FID9: value one pin header -> one header pin
Changed lines of the file:
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@@
 			)
 		)
-		(property "Value" "one pin header"
+		(property "Value" "one header pin"
 			(at 17.272 39.878 0)
 			(effects
@@
 			)
 		)
-		(property "Value" "one pin header"
+		(property "Value" "one header pin"
 			(at 17.272 74.168 0)
 			(effects
@@
 			)
 		)
-		(property "Value" "one pin header"
+		(property "Value" "one header pin"
 			(at 17.272 42.418 0)
 			(effects
@@
 			)
 		)
-		(property "Value" "one pin header"
+		(property "Value" "one header pin"
 			(at 17.272 75.438 0)
 			(effects
@@
 			)
 		)
-		(property "Value" "one pin header"
+		(property "Value" "one header pin"
 			(at 17.272 76.708 0)
 			(effects
@@
 			)
 		)
-		(property "Value" "one pin header"
+		(property "Value" "one header pin"
 			(at 17.272 41.148 0)
 			(effects
@@
 			)
 		)
-		(property "Value" "one pin header"
+		(property "Value" "one header pin"
 			(at 17.272 72.898 0)
 			(effects
@@
 			)
 		)
-		(property "Value" "one pin header"
+		(property "Value" "one header pin"
 			(at 17.272 38.608 0)
 			(effects

Commit message: update script
Parts:
- R3: value 2.5k -> 3.3k
Other:
- moved on the sheet: D3, R3
Changed lines of the file:
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@@
 	)
 	(junction
-		(at 73.66 110.49)
-		(diameter 0)
-		(color 0 0 0 0)
-	)
-	(junction
 		(at 261.62 60.96)
 		(diameter 0)
@@
 	)
 	(junction
+		(at 189.23 92.71)
+		(diameter 0)
+		(color 0 0 0 0)
+	)
+	(junction
 		(at 231.14 48.26)
 		(diameter 0)
@@
 	(wire
 		(pts
+			(xy 189.23 110.49) (xy 189.23 109.22)
+		)
+		(stroke
+			(width 0)
+			(type default)
+		)
+	)
+	(wire
+		(pts
 			(xy 251.46 35.56) (xy 261.62 35.56)
 		)
@@
 	(wire
 		(pts
-			(xy 73.66 110.49) (xy 73.66 116.84)
+			(xy 27.94 127) (xy 27.94 130.81)
 		)
 		(stroke
@@
 	(wire
 		(pts
-			(xy 27.94 127) (xy 27.94 130.81)
+			(xy 111.76 57.15) (xy 115.57 57.15)
 		)
 		(stroke
@@
 	(wire
 		(pts
-			(xy 111.76 57.15) (xy 115.57 57.15)
+			(xy 67.31 110.49) (xy 67.31 123.19)
 		)
 		(stroke
@@
 	(wire
 		(pts
-			(xy 67.31 110.49) (xy 67.31 123.19)
+			(xy 209.55 33.02) (xy 209.55 29.21)
 		)
 		(stroke
@@
 	(wire
 		(pts
-			(xy 209.55 33.02) (xy 209.55 29.21)
+			(xy 189.23 101.6) (xy 189.23 100.33)
 		)
 		(stroke
@@
 	(wire
 		(pts
-			(xy 90.17 116.84) (xy 88.9 116.84)
-		)
-		(stroke
-			(width 0)
-			(type default)
-		)
-	)
-	(wire
-		(pts
 			(xy 224.79 27.94) (xy 224.79 30.48)
 		)
@@
 	(wire
 		(pts
-			(xy 73.66 110.49) (xy 100.33 110.49)
+			(xy 67.31 110.49) (xy 100.33 110.49)
 		)
 		(stroke
@@
 	(wire
 		(pts
-			(xy 67.31 110.49) (xy 73.66 110.49)
-		)
-		(stroke
-			(width 0)
-			(type default)
-		)
-	)
-	(wire
-		(pts
 			(xy 80.01 17.78) (xy 80.01 31.75)
 		)
@@
 	(wire
 		(pts
-			(xy 196.85 92.71) (xy 200.66 92.71)
+			(xy 185.42 92.71) (xy 189.23 92.71)
 		)
 		(stroke
@@
 	(wire
 		(pts
+			(xy 189.23 92.71) (xy 200.66 92.71)
+		)
+		(stroke
+			(width 0)
+			(type default)
+		)
+	)
+	(wire
+		(pts
 			(xy 241.3 63.5) (xy 241.3 71.12)
 		)
@@
 	(global_label "14-3"
 		(shape input)
-		(at 196.85 92.71 180)
+		(at 185.42 92.71 180)
 		(fields_autoplaced yes)
 		(effects
@@
 		)
 		(property "Intersheetrefs" "${INTERSHEET_REFS}"
-			(at 188.6639 92.71 0)
+			(at 177.2339 92.71 0)
 			(effects
 				(font
@@
 	(symbol
 		(lib_id "Device:LED")
-		(at 77.47 116.84 180)
+		(at 189.23 96.52 90)
 		(unit 1)
 		(exclude_from_sim no)
@@
 		(dnp no)
 		(property "Reference" "D3"
-			(at 76.962 119.38 0)
+			(at 186.69 96.012 90)
 			(effects
 				(font
@@
 		)
 		(property "Value" "LED"
-			(at 79.248 121.158 0)
+			(at 187.96 98.044 90)
 			(effects
 				(font
@@
 		)
 		(property "Footprint" "218-pdb:LED_D3.0mm"
-			(at 77.47 116.84 0)
+			(at 189.23 96.52 0)
 			(effects
 				(font
@@
 		)
 		(property "Datasheet" "~"
-			(at 77.47 116.84 0)
+			(at 189.23 96.52 0)
 			(effects
 				(font
@@
 		)
 		(property "Description" "Light emitting diode"
-			(at 77.47 116.84 0)
+			(at 189.23 96.52 0)
 			(effects
 				(font
@@
 		)
 		(property "Sim.Pins" "1=K 2=A"
-			(at 77.47 116.84 0)
+			(at 189.23 96.52 0)
 			(effects
 				(font
@@
 		)
 		(property "Manufacturer_Name" ""
-			(at 77.47 116.84 0)
+			(at 189.23 96.52 0)
 			(effects
 				(font
@@
 		)
 		(property "digikey_part_number" ""
-			(at 77.47 116.84 0)
+			(at 189.23 96.52 0)
 			(effects
 				(font
@@
 		)
 		(property "mount_type" "tht"
-			(at 77.47 116.84 0)
+			(at 189.23 96.52 0)
 			(effects
 				(font
@@
 		)
 		(property "Part_Number" "3 mm diameter LED"
-			(at 77.47 116.84 90)
+			(at 189.23 96.52 90)
 			(effects
 				(font
@@
 	(symbol
 		(lib_id "power:GND")
-		(at 90.17 116.84 0)
+		(at 189.23 110.49 0)
 		(unit 1)
 		(exclude_from_sim no)
@@
 		(on_board yes)
 		(dnp no)
-		(fields_autoplaced yes)
 		(property "Reference" "#PWR020"
-			(at 90.17 123.19 0)
+			(at 189.23 116.84 0)
 			(effects
 				(font
@@
 		)
 		(property "Value" "GND"
-			(at 92.71 118.1099 0)
+			(at 189.992 113.03 0)
 			(effects
 				(font
@@
 		)
 		(property "Footprint" ""
-			(at 90.17 116.84 0)
+			(at 189.23 110.49 0)
 			(effects
 				(font
@@
 		)
 		(property "Datasheet" ""
-			(at 90.17 116.84 0)
+			(at 189.23 110.49 0)
 			(effects
 				(font
@@
 		)
 		(property "Description" "Power symbol creates a global label with name \"GND\" , ground"
-			(at 90.17 116.84 0)
+			(at 189.23 110.49 0)
 			(effects
 				(font
@@
 	(symbol
 		(lib_id "Device:R")
-		(at 85.09 116.84 90)
+		(at 189.23 105.41 0)
 		(unit 1)
 		(exclude_from_sim no)
@@
 		(dnp no)
 		(property "Reference" "R3"
-			(at 85.598 112.268 90)
+			(at 191.262 103.886 0)
 			(effects
 				(font
@@
 			)
 		)
-		(property "Value" "2.5k"
-			(at 87.122 114.3 90)
+		(property "Value" "3.3k"
+			(at 191.262 105.918 0)
 			(effects
 				(font
@@
 		)
 		(property "Footprint" "Resistor_THT:R_Axial_DIN0309_L9.0mm_D3.2mm_P2.54mm_Vertical"
-			(at 85.09 118.618 90)
+			(at 187.452 105.41 90)
 			(effects
 				(font
@@
 		)
 		(property "Datasheet" "~"
-			(at 85.09 116.84 0)
+			(at 189.23 105.41 0)
 			(effects
 				(font
@@
 		)
 		(property "Description" "Resistor"
-			(at 85.09 116.84 0)
+			(at 189.23 105.41 0)
 			(effects
 				(font
@@
 		)
 		(property "Manufacturer_Name" "any"
-			(at 85.09 116.84 0)
+			(at 189.23 105.41 0)
 			(effects
 				(font
@@
 		)
 		(property "digikey_part_number" "n/a"
-			(at 85.09 116.84 0)
+			(at 189.23 105.41 0)
 			(effects
 				(font
@@
 		)
 		(property "mount_type" "tht"
-			(at 85.09 116.84 0)
+			(at 189.23 105.41 0)
 			(effects
 				(font
@@
 		)
 		(property "Part_Number" "spdl"
-			(at 85.09 116.84 0)
+			(at 189.23 105.41 0)
 			(effects
 				(font
